File: breakout/gpioexp.kicad_pcb (KiCad board)
At the start: 2 copper layers, 20.3 x 33 mm, 9 parts, among them U1 AW9523B

Commit message: Rev c should be ready
Parts:
- renumbered C2 to C1, C1 to C2
Routing:
- net NRST: track 11.7 -> 12.6 mm
Changed lines of the file:
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@@
     (property "Sheetname" "")
     (attr smd)
-    (fp_text reference "C1" (at 0 -1.397) (layer "F.SilkS")
+    (fp_text reference "C2" (at 0 -1.397) (layer "F.SilkS")
       (effects (font (size 1 1) (thickness 0.15)))
     )
@@
     (property "Sheetname" "")
     (attr smd)
-    (fp_text reference "C2" (at -2.54 0) (layer "F.SilkS")
+    (fp_text reference "C1" (at -2.54 0) (layer "F.SilkS")
       (effects (font (size 1 1) (thickness 0.15)))
     )
@@
   (segment (start 135.86 104.14) (end 134.62 104.14) (width 0.2286) (layer "F.Cu") (net 6))
   (segment (start 139.5475 102.87) (end 137.13 102.87) (width 0.2286) (layer "F.Cu") (net 6))
-  (segment (start 147.67728 101.6) (end 149.86 101.6) (width 0.2286) (layer "F.Cu") (net 7))
-  (segment (start 142.99 94.0125) (end 142.99 96.91272) (width 0.2286) (layer "F.Cu") (net 7))
-  (segment (start 142.99 96.91272) (end 147.67728 101.6) (width 0.2286) (layer "F.Cu") (net 7))
-  (segment (start 142.49 94.0125) (end 142.49 97.972081) (width 0.2286) (layer "F.Cu") (net 8))
-  (segment (start 142.49 97.972081) (end 148.657919 104.14) (width 0.2286) (layer "F.Cu") (net 8))
-  (segment (start 148.657919 104.14) (end 149.86 104.14) (width 0.2286) (layer "F.Cu") (net 8))
-  (segment (start 139.77734 92.825) (end 135.736701 96.865639) (width 0.2286) (layer "F.Cu") (net 9))
-  (segment (start 135.736701 97.943299) (end 134.62 99.06) (width 0.2286) (layer "F.Cu") (net 9))
+  (segment (start 142.99 94.0125) (end 142.99 98.47) (width 0.2286) (layer "F.Cu") (net 7))
+  (segment (start 142.99 98.47) (end 146.12 101.6) (width 0.2286) (layer "F.Cu") (net 7))
+  (segment (start 146.12 101.6) (end 149.86 101.6) (width 0.2286) (layer "F.Cu") (net 7))
+  (segment (start 142.49 98.508124) (end 148.121876 104.14) (width 0.2286) (layer "F.Cu") (net 8))
+  (segment (start 148.121876 104.14) (end 149.86 104.14) (width 0.2286) (layer "F.Cu") (net 8))
+  (segment (start 142.49 94.0125) (end 142.49 98.508124) (width 0.2286) (layer "F.Cu") (net 8))
+  (segment (start 139.77734 92.825) (end 136.40117 96.20117) (width 0.2286) (layer "F.Cu") (net 9))
   (segment (start 140.3025 92.825) (end 139.77734 92.825) (width 0.2286) (layer "F.Cu") (net 9))
-  (segment (start 135.736701 96.865639) (end 135.736701 97.943299) (width 0.2286) (layer "F.Cu") (net 9))
+  (segment (start 134.62 99.06) (end 136.40117 97.27883) (width 0.2286) (layer "F.Cu") (net 9))
+  (segment (start 136.40117 97.27883) (end 136.40117 96.20117) (width 0.2286) (layer "F.Cu") (net 9))
   (segment (start 138.815 92.325) (end 134.62 96.52) (width 0.2286) (layer "F.Cu") (net 10))
   (segment (start 140.3025 92.325) (end 138.815 92.325) (width 0.2286) (layer "F.Cu") (net 10))
